Commit message: 增加模型

File: src/raspbot_description/urdf/omniwheel.urdf.xacro (robot description, xacro)
@@ -1,6 +1,6 @@
 <?xml version="1.0"?>
-<robot xmlns:xacro="http://ros.org/wiki/xacro" name="raspbot_wheel" >
-    <xacro:macro name="raspbot_wheel" params="wheel_prefix *joint_pose">
-        <link name="${wheel_prefix}_wheel_link">
+<robot xmlns:xacro="http://ros.org/wiki/xacro" name="raspbot_omniwheel" >
+    <xacro:macro name="raspbot_omniwheel" params="wheel_prefix *joint_pose">
+        <link name="${wheel_prefix}_omniwheel_link">
         	<inertial>
 				<mass value="0.167" />
@@ -11,5 +11,5 @@
                 <origin xyz="0 0 0" rpy="0 0 0" />
                 <geometry>
-                    <mesh filename="package://raspbot_description/meshes/wheel.dae" />
+                    <mesh filename="package://raspbot_description/meshes/omniwheel.dae" />
                 </geometry>
             </visual>
@@ -17,5 +17,5 @@
         <joint name="${wheel_prefix}_wheel" type="continuous">
             <parent link="base_link"/>
-            <child link="${wheel_prefix}_wheel_link"/>
+            <child link="${wheel_prefix}_omniwheel_link"/>
             <xacro:insert_block name="joint_pose"/>
             <axis xyz="0 1 0" rpy="0 0 0" />

File: src/raspbot_description/urdf/raspbot.urdf.xacro (robot description, xacro)
@@ -1,12 +1,91 @@
 <?xml version="1.0"?>
 <robot name="raspbot" xmlns:xacro="http://ros.org/wiki/xacro">
+    <xacro:property name="M_PI" value="3.1415916"/>
+    <xacro:include filename="$(find raspbot_description)/urdf/wheel.urdf.xacro" />
+    <xacro:include filename="$(find raspbot_description)/urdf/omniwheel.urdf.xacro" />
+    <xacro:include filename="$(find raspbot_description)/urdf/rplidar.urdf.xacro" />
+    <xacro:property name="base_footprint_offset" value="-0.049" />
+    <!-- Wheel Properties -->
+    <xacro:property name="wheel_length" value="0.027" />
+    <xacro:property name="wheel_radius" value="0.0335" />
+    <!-- Wheel Mounting Positions -->
+    <xacro:property name="wheeltrack" value="0.203" />
+    <xacro:property name="wheel_vertical_offset" value="0.0165" />
+    <xacro:property name="wheel_horizontal_offset" value="0.068" />
+    <!-- omniWheel Mounting Positions -->
+    <xacro:property name="omniwheel_x_offset" value="-0.0455" />
+    <xacro:property name="omniwheel_vertical_offset" value="-0.006" />
     <link name="base_link">
         <visual>
         <origin xyz="0 0 0" rpy="0 0 0" />
         <geometry>
-            <mesh filename="package://raspbot_description/meshes/baseH.dae" />
+            <mesh filename="package://raspbot_description/meshes/base.dae" />
         </geometry>
         </visual>
     </link>
-    <!-- <xacro:include filename="$(find husky_description)/urdf/wheel.urdf.xacro" /> -->
+    <link name="base_footprint"/>
+    <joint name="base_footprint_joint" type="fixed">
+        <origin xyz="0 0 ${base_footprint_offset}" rpy="0 0 0" />
+        <parent link="base_link" />
+        <child link="base_footprint" />
+    </joint>
+    <!--  wheel  -->
+    <xacro:raspbot_wheel wheel_prefix="left">
+        <origin xyz="${wheel_horizontal_offset} ${wheeltrack/2} ${-wheel_vertical_offset}" rpy="0 0 0" />
+    </xacro:raspbot_wheel>
+    <xacro:raspbot_wheel wheel_prefix="right">
+        <origin xyz="${wheel_horizontal_offset} ${-wheeltrack/2} ${-wheel_vertical_offset}" rpy="${M_PI} 0 0" />
+    </xacro:raspbot_wheel>
+    <!-- omniwheel -->
+    <xacro:raspbot_omniwheel wheel_prefix="rear">
+        <origin xyz="${omniwheel_x_offset} 0 ${omniwheel_vertical_offset}" rpy="0 0 ${M_PI}" />
+    </xacro:raspbot_omniwheel>
+    <xacro:rplidar frame="lidar_link" topic="scan" robot_namespace="$(arg robot_namespace)"/>
+    <joint name="base_lidar_joint" type="fixed">
+        <origin xyz="0.0693 0 0.0807" rpy="0 0 0" />
+        <parent link="base_link" />
+        <child link="lidar_link" />
+    </joint>
+    <!-- <link name="imu_link"/>
+    <joint name="base_footprint_joint" type="fixed">
+        <origin xyz="0 0 0" rpy="0 0 0" />
+        <parent link="base_link" />
+        <child link="imu_link" />
+    </joint> -->
+    <!--  gazebo  -->
+    <gazebo>
+        <plugin name="gazebo_ros_control" filename="libgazebo_ros_control.so">
+            <robotNamespace>$(arg robot_namespace)</robotNamespace>
+            <legacyModeNS>true</legacyModeNS>
+        </plugin>
+    </gazebo>
+    <!-- <gazebo>
+        <plugin name="imu_controller" filename="libhector_gazebo_ros_imu.so">
+            <robotNamespace>$(arg robot_namespace)</robotNamespace>
+            <updateRate>50.0</updateRate>
+            <bodyName>base_link</bodyName>
+            <topicName>imu/data</topicName>
+            <accelDrift>0.005 0.005 0.005</accelDrift>
+            <accelGaussianNoise>0.005 0.005 0.005</accelGaussianNoise>
+            <rateDrift>0.005 0.005 0.005 </rateDrift>
+            <rateGaussianNoise>0.005 0.005 0.005 </rateGaussianNoise>
+            <headingDrift>0.005</headingDrift>
+            <headingGaussianNoise>0.005</headingGaussianNoise>
+        </plugin>
+    </gazebo> -->
+  <!-- <gazebo>
+    <plugin name="gps_controller" filename="libhector_gazebo_ros_gps.so">
+      <robotNamespace>$(arg robot_namespace)</robotNamespace>
+      <updateRate>40</updateRate>
+      <bodyName>base_link</bodyName>
+      <frameId>base_link</frameId>
+      <topicName>navsat/fix</topicName>
+      <velocityTopicName>navsat/vel</velocityTopicName>
+      <referenceLatitude>49.9</referenceLatitude>
+      <referenceLongitude>8.9</referenceLongitude>
+      <referenceHeading>0</referenceHeading>
+      <referenceAltitude>0</referenceAltitude>
+      <drift>0.0001 0.0001 0.0001</drift>
+    </plugin>
+  </gazebo> -->
 </robot>

Commit message: gazebo

File: src/raspbot_description/urdf/omniwheel.urdf.xacro (robot description, xacro)
@@ -1,22 +1,77 @@
-<?xml version="1.0"?>
-<robot xmlns:xacro="http://ros.org/wiki/xacro" name="raspbot_omniwheel" >
-    <xacro:macro name="raspbot_omniwheel" params="wheel_prefix *joint_pose">
-        <link name="${wheel_prefix}_omniwheel_link">
-        	<inertial>
-				<mass value="0.167" />
-				<origin xyz="0 0 0" />
-				<inertia  ixx="0.02467" ixy="0" ixz="0" iyy="0.04411" iyz="0" izz="0.02467" />
-			</inertial>
+<robot name="raspbot_omniwheel" xmlns:xacro="http://ros.org/wiki/xacro"  >
+    <xacro:macro name="raspbot_omniwheel">
+        <!-- omniwheel part-->
+        <link name="omniwheel_part1_link">
+            <inertial>
+                <mass value="0.01" />
+                <origin xyz="0 0 0" />
+                <inertia ixx="0.001" ixy="0" ixz="0" iyy="0.001" iyz="0" izz="0.001" />
+            </inertial>
             <visual>
                 <origin xyz="0 0 0" rpy="0 0 0" />
                 <geometry>
-                    <mesh filename="package://raspbot_description/meshes/omniwheel.dae" />
+                    <mesh filename="package://raspbot_description/meshes/omniwheel_part1.dae" />
                 </geometry>
             </visual>
+            <collision>
+                <origin xyz="0 0 0" rpy="0 0 0" />
+                <geometry>
+                    <box size="0.039 0.033 0.002"/>
+                </geometry>
+            </collision>
         </link>
-        <joint name="${wheel_prefix}_wheel" type="continuous">
-            <parent link="base_link"/>
-            <child link="${wheel_prefix}_omniwheel_link"/>
-            <xacro:insert_block name="joint_pose"/>
+        <joint name="base_omniwheel_part1_joint" type="fixed">
+            <origin xyz="${omniwheel_x_offset} 0 ${omniwheel_vertical_offset}" rpy="0 0 0" />
+            <parent link="base_link" />
+            <child link="omniwheel_part1_link" />
+        </joint>
+        <link name="omniwheel_part2_link">
+            <inertial>
+                <mass value="0.04" />
+                <origin xyz="0 0 0" />
+                <inertia ixx="0.004" ixy="0" ixz="0" iyy="0.004" iyz="0" izz="0.004" />
+            </inertial>
+            <visual>
+                <origin xyz="0 0 0" rpy="0 0 0" />
+                <geometry>
+                    <mesh filename="package://raspbot_description/meshes/omniwheel_part2.dae" />
+                </geometry>
+            </visual>
+            <collision>
+                <origin xyz="0 0 0" rpy="0 0 0" />
+                <geometry>
+                    <cylinder length="0.01" radius="0.02" />
+                </geometry>
+            </collision>
+        </link>
+        <joint name="omniwheel_part1_2_joint" type="continuous">
+            <origin xyz="0 0 -0.01638" rpy="0 0 0" />
+            <parent link="omniwheel_part1_link" />
+            <child link="omniwheel_part2_link" />
+            <axis xyz="0 0 1" rpy="0 0 0" />
+        </joint>
+        <link name="omniwheel_part3_link">
+            <inertial>
+                <mass value="0.006" />
+                <origin xyz="0 0 0" />
+                <inertia ixx="0.001" ixy="0" ixz="0" iyy="0.001" iyz="0" izz="0.001" />
+            </inertial>
+            <visual>
+                <origin xyz="0 0 0" rpy="0 0 0" />
+                <geometry>
+                    <mesh filename="package://raspbot_description/meshes/omniwheel_part3.dae" />
+                </geometry>
+            </visual>
+            <collision>
+                <origin xyz="-0.015 0 0" rpy="0 0 0" />
+                <geometry>
+                    <cylinder length="0.025" radius="0.028" />
+                </geometry>
+            </collision>
+        </link>
+        <joint name="omniwheel_part2_3_joint" type="continuous">
+            <origin xyz="-0.015 0 -0.00718" rpy="0 0 0" />
+            <parent link="omniwheel_part2_link" />
+            <child link="omniwheel_part3_link" />
             <axis xyz="0 1 0" rpy="0 0 0" />
         </joint>

File: src/raspbot_description/urdf/raspbot.urdf.xacro (robot description, xacro)
@@ -1,9 +1,6 @@
 <?xml version="1.0"?>
 <robot name="raspbot" xmlns:xacro="http://ros.org/wiki/xacro">
+    <xacro:arg name="use_part_omni_model" default="true" />
     <xacro:property name="M_PI" value="3.1415916"/>
-    <xacro:include filename="$(find raspbot_description)/urdf/wheel.urdf.xacro" />
-    <xacro:include filename="$(find raspbot_description)/urdf/rplidar.urdf.xacro" />
-    <!-- The whole model can't simulate the omni model precisely -->
-    <!-- <xacro:include filename="$(find raspbot_description)/urdf/omniwheel.urdf.xacro" /> -->
     <!-- Base Size -->
     <xacro:property name="base_x_size" value="0.2" />
@@ -20,13 +17,16 @@
     <!-- omniWheel Mounting Positions -->
     <xacro:property name="omniwheel_x_offset" value="-0.053" />
-    <xacro:property name="omniwheel_vertical_offset" value="-0.01" />
+    <xacro:property name="omniwheel_vertical_offset" value="-0.011" />
     <!-- lidar Mounting Positions -->
     <xacro:property name="lidar_x_offset" value="0.06155" />
-     <xacro:property name="lidar_vertical_offset" value="0.081" />
+    <xacro:property name="lidar_vertical_offset" value="0.081" />
+    <xacro:include filename="$(find raspbot_description)/urdf/wheel.urdf.xacro" />
+    <xacro:include filename="$(find raspbot_description)/urdf/rplidar.urdf.xacro" />
+    <xacro:include filename="$(find raspbot_description)/urdf/omniwheel.urdf.xacro" />
     <link name="base_link">
         <visual>
             <origin xyz="0 0 0" rpy="0 0 0" />
             <geometry>
-                <mesh filename="package://raspbot_description/meshes/base1.dae" />
+                <mesh filename="package://raspbot_description/meshes/base.dae" />
             </geometry>
         </visual>
@@ -34,13 +34,13 @@
             <origin xyz="0 0 0" rpy="0 0 0" />
             <geometry>
-                <box size="0.01 0.01 0.01"/>
+                <box size="${base_x_size} ${base_y_size} ${base_z_size}"/>
             </geometry>
         </collision>
-        <!-- <collision>
+        <collision>
             <origin xyz="${base_x_size/2+0.00707} 0 0" rpy="0 0 0" />
             <geometry>
                 <box size="0.0141 ${base_y_size} ${base_z_size}"/>
             </geometry>
-        </collision> -->
+        </collision>
     </link>
     <link name="inertial_link">
@@ -48,5 +48,5 @@
             <mass value="1.5" />
             <origin xyz="0 0 0" />
-            <inertia ixx="0.06022" ixy="-0.002364" ixz="-0.01197" iyy="0.017386" iyz="-0.001544" izz="0.00296" />
+            <inertia ixx="0.15" ixy="0" ixz="0" iyy="0.15" iyz="0" izz="0.15" />
         </inertial>
     </link>
@@ -63,99 +63,38 @@
     </joint>
     <!--  wheel  -->
-    <!-- <xacro:raspbot_wheel wheel_prefix="left">
+    <xacro:raspbot_wheel wheel_prefix="left">
         <origin xyz="${wheel_horizontal_offset} ${wheeltrack/2} ${wheel_vertical_offset}" rpy="0 0 0" />
     </xacro:raspbot_wheel>
     <xacro:raspbot_wheel wheel_prefix="right">
         <origin xyz="${wheel_horizontal_offset} ${-wheeltrack/2} ${wheel_vertical_offset}" rpy="${M_PI} 0 0" />
-    </xacro:raspbot_wheel> -->
-    <!-- omniwheel part-->
-    <!-- <link name="omniwheel_part1_link">
-        <visual>
-            <origin xyz="0 0 0" rpy="0 0 0" />
-            <geometry>
-                <mesh filename="package://raspbot_description/meshes/omniwheel_part1.dae" />
-            </geometry>
-        </visual>
-    </link>
-    <joint name="base_omniwheel_part1_joint" type="fixed">
-        <origin xyz="${omniwheel_x_offset} 0 ${omniwheel_vertical_offset}" rpy="0 0 0" />
-        <parent link="base_link" />
-        <child link="omniwheel_part1_link" />
-    </joint> -->
-    <!-- <link name="omniwheel_part2_link">
-        <inertial>
-            <mass value="0.02" />
-            <origin xyz="0 0 0" />
-            <inertia ixx="0.001" ixy="0.001" ixz="0.001" iyy="0.001" iyz="0.001" izz="0.001" />
-        </inertial>
-        <visual>
-            <origin xyz="0 0 0" rpy="0 0 0" />
-            <geometry>
-                <mesh filename="package://raspbot_description/meshes/omniwheel_part2.dae" />
-            </geometry>
-        </visual>
-        <collision>
-            <origin xyz="0 0 0" rpy="0 0 0" />
-            <geometry>
-                <cylinder length="0.032" radius="0.028" />
-            </geometry>
-        </collision>
-    </link>
-    <joint name="omniwheel_part1_2_joint" type="continuous">
-        <origin xyz="0 0 -0.01638" rpy="0 0 0" />
-        <parent link="omniwheel_part1_link" />
-        <child link="omniwheel_part2_link" />
-        <axis xyz="0 0 1" rpy="0 0 0" />
-    </joint>
-    <link name="omniwheel_part3_link">
-        <visual>
-            <origin xyz="0 0 0" rpy="0 0 0" />
-            <geometry>
-                <mesh filename="package://raspbot_description/meshes/omniwheel_part3.dae" />
-            </geometry>
-        </visual>
-    </link>
-    <joint name="omniwheel_part2_3_joint" type="continuous">
-        <origin xyz="-0.015 0 -0.00718" rpy="0 0 0" />
-        <parent link="omniwheel_part2_link" />
-        <child link="omniwheel_part3_link" />
-        <axis xyz="0 1 0" rpy="0 0 0" />
-    </joint> -->
+    </xacro:raspbot_wheel>
     <!-- omniwheel -->
-    <!-- <xacro:raspbot_omniwheel wheel_prefix="rear">
-        <origin xyz="${omniwheel_x_offset} 0 ${omniwheel_vertical_offset}" rpy="0 0 ${M_PI}" />
-    </xacro:raspbot_omniwheel> -->
-    <!-- <xacro:rplidar frame="lidar_link" topic="scan" robot_namespace="$(arg robot_namespace)"/>
+    <xacro:raspbot_omniwheel />
+    <xacro:rplidar frame="lidar_link" topic="scan" robot_namespace="$(arg robot_namespace)"/>
     <joint name="base_lidar_joint" type="fixed">
         <origin xyz="${lidar_x_offset} 0 ${lidar_vertical_offset}" rpy="0 0 0" />
         <parent link="base_link" />
         <child link="lidar_link" />
-    </joint>  -->
-    <!-- <link name="imu_link"/>
+    </joint>
+    <link name="imu_link"/>
     <joint name="base_imu_joint" type="fixed">
         <origin xyz="0 0 0" rpy="0 0 0" />
         <parent link="base_link" />
         <child link="imu_link" />
-    </joint> -->
-    <link name="test_link">
-        <visual>
-            <origin xyz="0 0 0.08" rpy="${M_PI/2} 0 0" />
-            <geometry>
-                <cylinder length="${wheel_length}" radius="${wheel_radius}" />
-            </geometry>
-        </visual>
-        <collision>
-            <origin xyz="0 0 0" rpy="0 0 0" />
-            <geometry>
-                <cylinder length="${wheel_length}" radius="${wheel_radius}" />
-            </geometry>
-        </collision>
-    </link>
-    <joint name="base_test_joint" type="fixed">
-        <origin xyz="0 0 0.08" rpy="0 0 0" />
-        <parent link="base_link" />
-        <child link="test_link" />
     </joint>
     <!--  gazebo  -->
+    <!-- for all link -->
+    <gazebo>
+        <plugin name="gazebo_ros_control" filename="libgazebo_ros_control.so">
+            <robotNamespace>$(arg robot_namespace)</robotNamespace>
+            <legacyModeNS>true</legacyModeNS>
+        </plugin>
+    </gazebo>
+    <gazebo>
+        <plugin name="gazebo_ros_control" filename="libgazebo_ros_control.so">
+            <robotNamespace>$(arg robot_namespace)</robotNamespace>
+            <legacyModeNS>true</legacyModeNS>
+        </plugin>
+    </gazebo>
     <gazebo>
         <plugin name="gazebo_ros_control" filename="libgazebo_ros_control.so">

File: src/raspbot_description/urdf/rplidar.urdf.xacro (robot description, xacro)
@@ -30,9 +30,9 @@
     <link name="${frame}">
       <inertial>
-        <mass value="1.1" />
+        <mass value="0.017" />
         <origin xyz="0 0 0" />
-        <inertia ixx="${0.0833333 * 1.1 * (0.102*0.102 + 0.152*0.152)}" ixy="0.0" ixz="0.0"
-          iyy="${0.0833333 * 1.1 * (0.105*0.105 + 0.152*0.152)}" iyz="0.0"
-          izz="${0.0833333 * 1.1 * (0.105*0.105 + 0.102*0.102)}" />
+        <inertia ixx="0.0017" ixy="0.0" ixz="0.0"
+          iyy="0.0017" iyz="0.0"
+          izz="0.0017" />
       </inertial>
       <visual>

File: src/raspbot_description/urdf/wheel.urdf.xacro (robot description, xacro)
@@ -4,7 +4,7 @@
         <link name="${wheel_prefix}_wheel_link">
         	<inertial>
-				<mass value="0.167" />
+				<mass value="0.034" />
 				<origin xyz="0 0 0" />
-				<inertia  ixx="0.001" ixy="0" ixz="0" iyy="0.001" iyz="0" izz="0.001" />
+				<inertia  ixx="0.0005" ixy="0" ixz="0" iyy="0.0005" iyz="0" izz="0.0005" />.01
 			</inertial>
             <visual>
