Commit message: change gazebo params

File: src/raspbot_description/urdf/omniwheel.urdf.xacro (robot description, xacro)
@@ -6,5 +6,5 @@
                 <mass value="0.01" />
                 <origin xyz="0 0 0" />
-                <inertia ixx="0.001" ixy="0" ixz="0" iyy="0.001" iyz="0" izz="0.001" />
+                <inertia ixx="0.01" ixy="0" ixz="0" iyy="0.01" iyz="0" izz="0.01" />
             </inertial>
             <visual>
@@ -28,7 +28,9 @@
         <link name="omniwheel_part2_link">
             <inertial>
-                <mass value="0.04" />
+                <mass value="1" />
                 <origin xyz="0 0 0" />
-                <inertia ixx="0.004" ixy="0" ixz="0" iyy="0.004" iyz="0" izz="0.004" />
+                <inertia ixx="1" ixy="0" ixz="0"
+                    iyy="1" iyz="0"
+                    izz="1" />
             </inertial>
             <visual>
@@ -53,7 +55,9 @@
         <link name="omniwheel_part3_link">
             <inertial>
-                <mass value="0.006" />
+                <mass value="0.01" />
                 <origin xyz="0 0 0" />
-                <inertia ixx="0.001" ixy="0" ixz="0" iyy="0.001" iyz="0" izz="0.001" />
+                <inertia ixx="0.001" ixy="0" ixz="0"
+                iyy="0.001" iyz="0"
+                izz="0.001" />
             </inertial>
             <visual>
@@ -76,4 +80,18 @@
             <axis xyz="0 1 0" rpy="0 0 0" />
         </joint>
+        <gazebo reference="omniwheel_part2_link">
+			<mu1 value="0.01"/>
+			<mu2 value="0.01"/>
+			<kp value="10000000.0" />
+			<kd value="1.0" />
+			<fdir1 value="1 0 0"/>
+		</gazebo>
+        <gazebo reference="omniwheel_part3_link">
+			<mu1 value="0.1"/>
+			<mu2 value="0.1"/>
+			<kp value="10000000.0" />
+			<kd value="1.0" />
+			<fdir1 value="1 0 0"/>
+		</gazebo>
     </xacro:macro>
 </robot>

File: src/raspbot_description/urdf/raspbot.urdf.xacro (robot description, xacro)
@@ -7,8 +7,8 @@
     <xacro:property name="base_y_size" value="0.16" />
     <xacro:property name="base_z_size" value="0.07" />
-    <xacro:property name="base_footprint_offset" value="-0.049" />
+    <xacro:property name="base_footprint_offset" value="0.049" />
     <!-- Wheel Properties -->
     <xacro:property name="wheel_length" value="0.027" />
-    <xacro:property name="wheel_radius" value="0.0335" />
+    <xacro:property name="wheel_radius" value="0.0325" />
     <!-- Wheel Mounting Positions -->
     <xacro:property name="wheeltrack" value="0.203" />
@@ -24,5 +24,13 @@
     <xacro:include filename="$(find raspbot_description)/urdf/rplidar.urdf.xacro" />
     <xacro:include filename="$(find raspbot_description)/urdf/omniwheel.urdf.xacro" />
+    <link name="base_footprint"/>
     <link name="base_link">
+        <inertial>
+            <mass value="2" />
+            <origin xyz="0 0 0" />
+            <inertia ixx="0.2" ixy="0" ixz="0"
+                iyy="0.2" iyz="0"
+                izz="0.2" />
+        </inertial>
         <visual>
             <origin xyz="0 0 0" rpy="0 0 0" />
@@ -34,44 +42,48 @@
             <origin xyz="0 0 0" rpy="0 0 0" />
             <geometry>
-                <box size="${base_x_size} ${base_y_size} ${base_z_size}"/>
+                <box size="0.2 0.16 0.007"/>
+                <!-- <box size="${base_x_size} ${base_y_size} ${base_z_size}"/> -->
             </geometry>
         </collision>
         <collision>
-            <origin xyz="${base_x_size/2+0.00707} 0 0" rpy="0 0 0" />
+            <origin xyz="0.10857 0 0" rpy="0 0 0" />
+            <!-- <origin xyz="${base_x_size/2+0.00707} 0 0" rpy="0 0 0" /> -->
             <geometry>
-                <box size="0.0141 ${base_y_size} ${base_z_size}"/>
+                <!-- <box size="0.0141 ${base_y_size} ${base_z_size}"/> -->
+                <box size="0.0141 0.16 0.007"/>
             </geometry>
         </collision>
     </link>
-    <link name="inertial_link">
-        <inertial>
-            <mass value="1.5" />
-            <origin xyz="0 0 0" />
-            <inertia ixx="0.15" ixy="0" ixz="0" iyy="0.15" iyz="0" izz="0.15" />
-        </inertial>
-    </link>
-    <joint name="inertial_joint" type="fixed">
-        <origin xyz="0 0 0" rpy="0 0 0" />
-        <parent link="base_link" />
-        <child link="inertial_link" />
-    </joint>
-    <link name="base_footprint"/>
     <joint name="base_footprint_joint" type="fixed">
         <origin xyz="0 0 ${base_footprint_offset}" rpy="0 0 0" />
-        <parent link="base_link" />
-        <child link="base_footprint" />
+        <parent link="base_footprint" />
+        <child link="base_link" />
     </joint>
     <!--  wheel  -->
     <xacro:raspbot_wheel wheel_prefix="left">
         <origin xyz="${wheel_horizontal_offset} ${wheeltrack/2} ${wheel_vertical_offset}" rpy="0 0 0" />
+        <axis xyz="0 1 0" rpy="0 0 0" />
     </xacro:raspbot_wheel>
     <xacro:raspbot_wheel wheel_prefix="right">
         <origin xyz="${wheel_horizontal_offset} ${-wheeltrack/2} ${wheel_vertical_offset}" rpy="${M_PI} 0 0" />
+        <axis xyz="0 -1 0" rpy="0 0 0" />
     </xacro:raspbot_wheel>
     <!-- omniwheel -->
     <xacro:raspbot_omniwheel />
     <xacro:rplidar frame="lidar_link" topic="scan" robot_namespace="$(arg robot_namespace)"/>
+    <!-- <xacro:rplidar>
+        frame="lidar_link"
+        topic="scan"
+        min_angle="-2.35619"
+        max_angle="-2.35619"
+        min_range="-2.35619"
+        max_range="-2.35619"
+        sample_size="-2.35619"
+        update_rate="10.0"
+        robot_namespace="$(arg robot_namespace)"
+    </xacro:rplidar> -->
     <joint name="base_lidar_joint" type="fixed">
-        <origin xyz="${lidar_x_offset} 0 ${lidar_vertical_offset}" rpy="0 0 0" />
+        <!-- <origin xyz="${lidar_x_offset} 0 ${lidar_vertical_offset}" rpy="0 0 0" /> -->
+        <origin xyz="0.06155 0.0 0.081" rpy="0 0 0" />
         <parent link="base_link" />
         <child link="lidar_link" />
@@ -84,5 +96,4 @@
     </joint>
     <!--  gazebo  -->
-    <!-- for all link -->
     <gazebo>
         <plugin name="gazebo_ros_control" filename="libgazebo_ros_control.so">
@@ -91,18 +102,26 @@
         </plugin>
     </gazebo>
-    <gazebo>
-        <plugin name="gazebo_ros_control" filename="libgazebo_ros_control.so">
-            <robotNamespace>$(arg robot_namespace)</robotNamespace>
-            <legacyModeNS>true</legacyModeNS>
-        </plugin>
-    </gazebo>
-    <gazebo>
-        <plugin name="gazebo_ros_control" filename="libgazebo_ros_control.so">
-            <robotNamespace>$(arg robot_namespace)</robotNamespace>
-            <legacyModeNS>true</legacyModeNS>
-        </plugin>
-    </gazebo>
+    <!-- <gazebo reference="imu_link">
+        <gravity>true</gravity>
+        <sensor name="imu_sensor" type="imu">
+            <always_on>true</always_on>
+            <update_rate>100</update_rate>
+            <visualize>true</visualize>
+            <topic>__default_topic__</topic>
+            <plugin filename="libgazebo_ros_imu_sensor.so" name="imu_plugin">
+                <topicName>imu</topicName>
+                <bodyName>imu_link</bodyName>
+                <updateRateHZ>10.0</updateRateHZ>
+                <gaussianNoise>0.005</gaussianNoise>
+                <xyzOffset>0 0 0</xyzOffset>
+                <rpyOffset>0 0 0</rpyOffset>
+                <frameName>imu_link</frameName>
+                <initialOrientationAsReference>false</initialOrientationAsReference>
+            </plugin>
+            <pose>0 0 0 0 0 0</pose>
+        </sensor>
+    </gazebo>   -->
     <!-- <gazebo>
-        <plugin name="imu_controller" filename="libhector_gazebo_ros_imu.so">
+        <plugin name="imu_link" filename="libhector_gazebo_ros_imu.so">
             <robotNamespace>$(arg robot_namespace)</robotNamespace>
             <updateRate>50.0</updateRate>
@@ -117,18 +136,40 @@
         </plugin>
     </gazebo> -->
-  <!-- <gazebo>
-    <plugin name="gps_controller" filename="libhector_gazebo_ros_gps.so">
-      <robotNamespace>$(arg robot_namespace)</robotNamespace>
-      <updateRate>40</updateRate>
-      <bodyName>base_link</bodyName>
-      <frameId>base_link</frameId>
-      <topicName>navsat/fix</topicName>
-      <velocityTopicName>navsat/vel</velocityTopicName>
-      <referenceLatitude>49.9</referenceLatitude>
-      <referenceLongitude>8.9</referenceLongitude>
-      <referenceHeading>0</referenceHeading>
-      <referenceAltitude>0</referenceAltitude>
-      <drift>0.0001 0.0001 0.0001</drift>
-    </plugin>
-  </gazebo> -->
+    <!-- <gazebo>
+        <plugin name="gps_controller" filename="libhector_gazebo_ros_gps.so">
+            <robotNamespace>$(arg robot_namespace)</robotNamespace>
+            <updateRate>40</updateRate>
+            <bodyName>base_link</bodyName>
+            <frameId>base_link</frameId>
+            <topicName>navsat/fix</topicName>
+            <velocityTopicName>navsat/vel</velocityTopicName>
+            <referenceLatitude>49.9</referenceLatitude>
+            <referenceLongitude>8.9</referenceLongitude>
+            <referenceHeading>0</referenceHeading>
+            <referenceAltitude>0</referenceAltitude>
+            <drift>0.0001 0.0001 0.0001</drift>
+        </plugin>
+    </gazebo> -->
+    <!-- <gazebo>
+        <plugin name="differential_drive_controller" filename="libgazebo_ros_diff_drive.so">
+            <updateRate>50</updateRate>
+            <leftJoint>left_wheel</leftJoint>
+            <rightJoint>right_wheel</rightJoint>
+            <wheelSeparation>0.203</wheelSeparation>
+            <wheelDiameter>0.0325</wheelDiameter>
+            <wheelAcceleration>1.0</wheelAcceleration>
+            <wheelTorque>100</wheelTorque>
+            <commandTopic>cmd_vel</commandTopic>
+            <odometryTopic>odom</odometryTopic>
+            <odometryFrame>odom</odometryFrame>
+            <robotBaseFrame>base_link</robotBaseFrame>
+            <odometrySource>world</odometrySource>
+            <publishWheelTF>false</publishWheelTF>
+            <publishOdomTF>true</publishOdomTF>
+            <publishTf>true</publishTf>
+            <publishWheelJointState>false</publishWheelJointState>
+            <legacyMode>false</legacyMode>
+            <rosDebugLevel>na</rosDebugLevel>
+        </plugin>
+    </gazebo> -->
 </robot>

File: src/raspbot_description/urdf/rplidar.urdf.xacro (robot description, xacro)
@@ -1,28 +1,3 @@
 <?xml version="1.0"?>
-<!--
-Copyright (c) 2013, Goncalo Cabrita, ISR University of Coimbra
-Copyright (c) 2014, 2015 Clearpath Robotics
-All rights reserved.
-Redistribution and use in source and binary forms, with or without
-modification, are permitted provided that the following conditions are met:
-    * Redistributions of source code must retain the above copyright
-      notice, this list of conditions and the following disclaimer.
-    * Redistributions in binary form must reproduce the above copyright
-      notice, this list of conditions and the following disclaimer in the
-      documentation and/or other materials provided with the distribution.
-    * Neither the name of Clearpath Robotics nor the
-      names of its contributors may be used to endorse or promote products
-      derived from this software without specific prior written permission.
-THIS SOFTWARE IS PROVIDED BY THE COPYRIGHT HOLDERS AND CONTRIBUTORS "AS IS" AND
-ANY EXPRESS OR IMPLIED WARRANTIES, INCLUDING, BUT NOT LIMITED TO, THE IMPLIED
-WARRANTIES OF MERCHANTABILITY AND FITNESS FOR A PARTICULAR PURPOSE ARE
-DISCLAIMED. IN NO EVENT SHALL THE COPYRIGHT HOLDERS BE LIABLE FOR ANY
-DIRECT, INDIRECT, INCIDENTAL, SPECIAL, EXEMPLARY, OR CONSEQUENTIAL DAMAGES
-(INCLUDING, BUT NOT LIMITED TO, PROCUREMENT OF SUBSTITUTE GOODS OR SERVICES;
-LOSS OF USE, DATA, OR PROFITS; OR BUSINESS INTERRUPTION) HOWEVER CAUSED AND
-ON ANY THEORY OF LIABILITY, WHETHER IN CONTRACT, STRICT LIABILITY, OR TORT
-(INCLUDING NEGLIGENCE OR OTHERWISE) ARISING IN ANY WAY OUT OF THE USE OF THIS
-SOFTWARE, EVEN IF ADVISED OF THE POSSIBILITY OF SUCH DAMAGE.
--->
 <robot xmlns:xacro="http://www.ros.org/wiki/xacro">
   <xacro:macro name="rplidar" params="frame:=laser topic:=scan sample_size:=720 update_rate:=50
@@ -30,9 +5,9 @@
     <link name="${frame}">
       <inertial>
-        <mass value="0.017" />
+        <mass value="0.17" />
         <origin xyz="0 0 0" />
-        <inertia ixx="0.0017" ixy="0.0" ixz="0.0"
-          iyy="0.0017" iyz="0.0"
-          izz="0.0017" />
+        <inertia ixx="0.17" ixy="0.0" ixz="0.0"
+          iyy="0.17" iyz="0.0"
+          izz="0.17" />
       </inertial>
       <visual>

File: src/raspbot_description/urdf/wheel.urdf.xacro (robot description, xacro)
@@ -1,10 +1,12 @@
 <?xml version="1.0"?>
 <robot xmlns:xacro="http://ros.org/wiki/xacro" name="raspbot_wheel" >
-    <xacro:macro name="raspbot_wheel" params="wheel_prefix *joint_pose">
+    <xacro:macro name="raspbot_wheel" params="wheel_prefix *joint_pose  *axis">
         <link name="${wheel_prefix}_wheel_link">
         	<inertial>
 				<mass value="0.034" />
 				<origin xyz="0 0 0" />
-				<inertia  ixx="0.0005" ixy="0" ixz="0" iyy="0.0005" iyz="0" izz="0.0005" />.01
+				<inertia  ixx="0.034" ixy="0" ixz="0"
+					iyy="0.034" iyz="0"
+					izz="0.034" />
 			</inertial>
             <visual>
@@ -25,5 +27,5 @@
             <child link="${wheel_prefix}_wheel_link"/>
             <xacro:insert_block name="joint_pose"/>
-            <axis xyz="0 1 0" rpy="0 0 0" />
+            <xacro:insert_block name="axis"/>
         </joint>
 		<gazebo reference="${wheel_prefix}_wheel_link">
@@ -36,10 +38,11 @@
 		<transmission name="${wheel_prefix}_wheel_trans" type="SimpleTransmission">
 			<type>transmission_interface/SimpleTransmission</type>
-			<actuator name="${wheel_prefix}_wheel_motor">
-				<mechanicalReduction>1</mechanicalReduction>
-			</actuator>
 			<joint name="${wheel_prefix}_wheel">
 				<hardwareInterface>hardware_interface/VelocityJointInterface</hardwareInterface>
 			</joint>
+			<actuator name="${wheel_prefix}_wheel_motor">
+				<hardwareInterface>hardware_interface/VelocityJointInterface</hardwareInterface>
+				<mechanicalReduction>1</mechanicalReduction>
+			</actuator>
 		</transmission>
     </xacro:macro>

Commit message: change params

File: src/raspbot_description/urdf/omniwheel.urdf.xacro (robot description, xacro)
@@ -4,7 +4,9 @@
         <link name="omniwheel_part1_link">
             <inertial>
-                <mass value="0.01" />
+                <mass value="0.016" />
                 <origin xyz="0 0 0" />
-                <inertia ixx="0.01" ixy="0" ixz="0" iyy="0.01" iyz="0" izz="0.01" />
+                <inertia ixx="2.23E-06" ixy="0" ixz="0"
+                    iyy="3.77E-06" iyz="0"
+                    izz="1.568E-06" />
             </inertial>
             <visual>
@@ -28,9 +30,12 @@
         <link name="omniwheel_part2_link">
             <inertial>
-                <mass value="1" />
-                <origin xyz="0 0 0" />
-                <inertia ixx="1" ixy="0" ixz="0"
-                    iyy="1" iyz="0"
-                    izz="1" />
+                <mass value="0.031" />
+                <origin xyz="-0.0035 0 0.007" />
+                <!-- <inertia ixx="3.91E-07" ixy="0" ixz="0"
+                    iyy="4.709E-07" iyz="0"
+                    izz="3.97E-07" /> -->
+                <inertia ixx="0.031" ixy="0" ixz="0"
+                    iyy="0.031" iyz="0"
+                    izz="0.031" />
             </inertial>
             <visual>
@@ -55,9 +60,9 @@
         <link name="omniwheel_part3_link">
             <inertial>
-                <mass value="0.01" />
+                <mass value="0.02" />
                 <origin xyz="0 0 0" />
-                <inertia ixx="0.001" ixy="0" ixz="0"
-                iyy="0.001" iyz="0"
-                izz="0.001" />
+                <inertia ixx="1.504E-06" ixy="0" ixz="0"
+                iyy="1.07E-06" iyz="0"
+                izz="1.07E-06" />
             </inertial>
             <visual>
@@ -81,6 +86,6 @@
         </joint>
         <gazebo reference="omniwheel_part2_link">
-			<mu1 value="0.01"/>
-			<mu2 value="0.01"/>
+			<mu1 value="0.5"/>
+			<mu2 value="0.5"/>
 			<kp value="10000000.0" />
 			<kd value="1.0" />
@@ -88,6 +93,6 @@
 		</gazebo>
         <gazebo reference="omniwheel_part3_link">
-			<mu1 value="0.1"/>
-			<mu2 value="0.1"/>
+			<mu1 value="1"/>
+			<mu2 value="1"/>
 			<kp value="10000000.0" />
 			<kd value="1.0" />

File: src/raspbot_description/urdf/raspbot.urdf.xacro (robot description, xacro)
@@ -27,9 +27,20 @@
     <link name="base_link">
         <inertial>
+            <!-- <mass value="2.8" /> -->
+            <!-- <mass value="1.5" /> -->
             <mass value="1.5" />
-            <origin xyz="0.0405 0 -0.0227" />
-            <inertia ixx="6.732188E-03" ixy="-5.9717E-05" ixz="-1.68616E-04"
+            <origin xyz="0.04 0.000 -0.00225" />
+            <!-- <inertia ixx="6.732188E-03" ixy="-5.9717E-05" ixz="-1.68616E-04"
                 iyy="1.002365E-02" iyz="1.51049E-04"
-                izz="4.991390E-03" />
+                izz="4.991390E-03" /> -->
+            <!-- <inertia ixx="1.2650E-02" ixy="-1.1198E-04" ixz="-2.94157E-04"
+                iyy="1.8646767E-02" iyz="2.31768E-04"
+                izz="9.173871E-03" />     -->
+            <!-- <inertia ixx="2.2592E-02" ixy="-1.9999E-04" ixz="-5.25345E-04"
+                iyy="3.3301E-02" iyz="4.13922E-04"
+                izz="1.6383935E-02" />   -->
+            <inertia ixx="1.5" ixy="0" ixz="0"
+                iyy="1.5" iyz="0"
+                izz="1.5" />
         </inertial>
         <visual>
@@ -68,21 +79,20 @@
     <!-- omniwheel -->
     <xacro:raspbot_omniwheel />
-    <xacro:rplidar frame="lidar_link" topic="scan" robot_namespace="$(arg robot_namespace)"/>
-    <!-- <xacro:rplidar>
+    <!-- <xacro:rplidar frame="lidar_link" topic="scan" robot_namespace="$(arg robot_namespace)"/> -->
+    <!-- <xacro:rplidar
         frame="lidar_link"
         topic="scan"
-        min_angle="-2.35619"
-        max_angle="-2.35619"
-        min_range="-2.35619"
-        max_range="-2.35619"
-        sample_size="-2.35619"
-        update_rate="10.0"
-        robot_namespace="$(arg robot_namespace)"
-    </xacro:rplidar> -->
-    <joint name="base_lidar_joint" type="fixed">
+        min_angle="${-M_PI}"
+        max_angle="${M_PI}"
+        min_range="0.15"
+        max_range="12"
+        sample_size="360"
+        update_rate="5.5"
+        robot_namespace="$(arg robot_namespace)" /> -->
+    <!-- <joint name="base_lidar_joint" type="fixed">
         <origin xyz="${lidar_x_offset} 0 ${lidar_vertical_offset}" rpy="0 0 0" />
         <parent link="base_link" />
         <child link="lidar_link" />
-    </joint>
+    </joint>  -->
     <link name="imu_link"/>
     <joint name="base_imu_joint" type="fixed">

File: src/raspbot_description/urdf/rplidar.urdf.xacro (robot description, xacro)
@@ -6,8 +6,8 @@
       <inertial>
         <mass value="0.17" />
-        <origin xyz="0 0 0" />
-        <inertia ixx="0.17" ixy="0.0" ixz="0.0"
-          iyy="0.17" iyz="0.0"
-          izz="0.17" />
+        <origin xyz="-0.01 0 -0.01" />
+        <inertia ixx="1.38228E-04" ixy="-0.616E-06" ixz="1.219E-06"
+          iyy="1.57876E-04" iyz="-2.1783E-05"
+          izz="6.8763E-05" />
       </inertial>
       <visual>

File: src/raspbot_description/urdf/wheel.urdf.xacro (robot description, xacro)
@@ -4,9 +4,9 @@
         <link name="${wheel_prefix}_wheel_link">
         	<inertial>
-				<mass value="0.034" />
+				<mass value="0.04" />
 				<origin xyz="0 0 0" />
-				<inertia  ixx="0.034" ixy="0" ixz="0"
-					iyy="0.034" iyz="0"
-					izz="0.034" />
+				<inertia  ixx="0.04" ixy="0" ixz="0"
+					iyy="0.04" iyz="0"
+					izz="0.04" />
 			</inertial>
             <visual>
