Commit message: add dae model

File: src/raspbot_description/urdf/raspbot.urdf.xacro (robot description, xacro)
@@ -5,5 +5,5 @@
         <origin xyz="0 0 0" rpy="0 0 0" />
         <geometry>
-            <mesh filename="package://raspbot_description/meshes/rplidar.dae" />
+            <mesh filename="package://raspbot_description/meshes/baseH.dae" />
         </geometry>
         </visual>

Commit message: change model and params

File: src/raspbot_description/urdf/raspbot.urdf.xacro (robot description, xacro)
@@ -11,9 +11,9 @@
     <!-- Wheel Mounting Positions -->
     <xacro:property name="wheeltrack" value="0.203" />
-    <xacro:property name="wheel_vertical_offset" value="0.0165" />
-    <xacro:property name="wheel_horizontal_offset" value="0.068" />
+    <xacro:property name="wheel_vertical_offset" value="-0.0145" />
+    <xacro:property name="wheel_horizontal_offset" value="0.0769" />
     <!-- omniWheel Mounting Positions -->
     <xacro:property name="omniwheel_x_offset" value="-0.0455" />
-    <xacro:property name="omniwheel_vertical_offset" value="-0.006" />
+    <xacro:property name="omniwheel_vertical_offset" value="-0.01" />
     <link name="base_link">
         <visual>
@@ -32,8 +32,8 @@
     <!--  wheel  -->
     <xacro:raspbot_wheel wheel_prefix="left">
-        <origin xyz="${wheel_horizontal_offset} ${wheeltrack/2} ${-wheel_vertical_offset}" rpy="0 0 0" />
+        <origin xyz="${wheel_horizontal_offset} ${wheeltrack/2} ${wheel_vertical_offset}" rpy="0 0 0" />
     </xacro:raspbot_wheel>
     <xacro:raspbot_wheel wheel_prefix="right">
-        <origin xyz="${wheel_horizontal_offset} ${-wheeltrack/2} ${-wheel_vertical_offset}" rpy="${M_PI} 0 0" />
+        <origin xyz="${wheel_horizontal_offset} ${-wheeltrack/2} ${wheel_vertical_offset}" rpy="${M_PI} 0 0" />
     </xacro:raspbot_wheel>
     <!-- omniwheel -->
@@ -43,5 +43,5 @@
     <xacro:rplidar frame="lidar_link" topic="scan" robot_namespace="$(arg robot_namespace)"/>
     <joint name="base_lidar_joint" type="fixed">
-        <origin xyz="0.0693 0 0.0807" rpy="0 0 0" />
+        <origin xyz="0.0705 0 0.0807" rpy="0 0 0" />
         <parent link="base_link" />
         <child link="lidar_link" />

Commit message: gazebo

File: src/raspbot_description/urdf/raspbot.urdf.xacro (robot description, xacro)
@@ -16,11 +16,26 @@
     <xacro:property name="omniwheel_x_offset" value="-0.0455" />
     <xacro:property name="omniwheel_vertical_offset" value="-0.01" />
+    <!-- lidar Mounting Positions -->
+    <xacro:property name="lidar_x_offset" value="0.0705" />
+    <xacro:property name="lidar_vertical_offset" value="0.0807" />
     <link name="base_link">
         <visual>
-        <origin xyz="0 0 0" rpy="0 0 0" />
-        <geometry>
-            <mesh filename="package://raspbot_description/meshes/base.dae" />
-        </geometry>
+            <origin xyz="0 0 0" rpy="0 0 0" />
+            <geometry>
+                <mesh filename="package://raspbot_description/meshes/base.dae" />
+            </geometry>
         </visual>
+        <collision>
+            <origin xyz="${( husky_front_bumper_extend - husky_rear_bumper_extend ) / 2.0} 0 ${base_z_size/4}" rpy="0 0 0" />
+            <geometry>
+                <box size="${ base_x_size + husky_front_bumper_extend + husky_rear_bumper_extend } ${base_y_size} ${base_z_size/2}"/>
+            </geometry>
+        </collision>
+        <collision>
+            <origin xyz="0 0 ${base_z_size*3/4-0.01}" rpy="0 0 0" />
+            <geometry>
+                <box size="${base_x_size*4/5} ${base_y_size} ${base_z_size/2-0.02}"/>
+            </geometry>
+        </collision>
     </link>
     <link name="base_footprint"/>
@@ -43,5 +58,5 @@
     <xacro:rplidar frame="lidar_link" topic="scan" robot_namespace="$(arg robot_namespace)"/>
     <joint name="base_lidar_joint" type="fixed">
-        <origin xyz="0.0705 0 0.0807" rpy="0 0 0" />
+        <origin xyz="${lidar_x_offset} 0 ${lidar_vertical_offset}" rpy="0 0 0" />
         <parent link="base_link" />
         <child link="lidar_link" />

File: src/raspbot_description/urdf/wheel.urdf.xacro (robot description, xacro)
@@ -21,4 +21,20 @@
             <axis xyz="0 1 0" rpy="0 0 0" />
         </joint>
+		<gazebo reference="${wheel_prefix}_wheel_link">
+			<mu1 value="1.0"/>
+			<mu2 value="1.0"/>
+			<kp value="10000000.0" />
+			<kd value="1.0" />
+			<fdir1 value="1 0 0"/>
+		</gazebo>
+		<transmission name="${wheel_prefix}_wheel_trans" type="SimpleTransmission">
+			<type>transmission_interface/SimpleTransmission</type>
+			<actuator name="${wheel_prefix}_wheel_motor">
+				<mechanicalReduction>1</mechanicalReduction>
+			</actuator>
+			<joint name="${wheel_prefix}_wheel">
+				<hardwareInterface>hardware_interface/VelocityJointInterface</hardwareInterface>
+			</joint>
+		</transmission>
     </xacro:macro>
 </robot>

Commit message: gazebo simulate

File: src/raspbot_description/urdf/raspbot.urdf.xacro (robot description, xacro)
@@ -3,6 +3,11 @@
     <xacro:property name="M_PI" value="3.1415916"/>
     <xacro:include filename="$(find raspbot_description)/urdf/wheel.urdf.xacro" />
-    <xacro:include filename="$(find raspbot_description)/urdf/omniwheel.urdf.xacro" />
     <xacro:include filename="$(find raspbot_description)/urdf/rplidar.urdf.xacro" />
+    <!-- The whole model can't simulate the omni model precisely -->
+    <!-- <xacro:include filename="$(find raspbot_description)/urdf/omniwheel.urdf.xacro" /> -->
+    <!-- Base Size -->
+    <xacro:property name="base_x_size" value="0.2" />
+    <xacro:property name="base_y_size" value="0.16" />
+    <xacro:property name="base_z_size" value="0.07" />
     <xacro:property name="base_footprint_offset" value="-0.049" />
     <!-- Wheel Properties -->
@@ -12,31 +17,43 @@
     <xacro:property name="wheeltrack" value="0.203" />
     <xacro:property name="wheel_vertical_offset" value="-0.0145" />
-    <xacro:property name="wheel_horizontal_offset" value="0.0769" />
+    <xacro:property name="wheel_horizontal_offset" value="0.068" />
     <!-- omniWheel Mounting Positions -->
-    <xacro:property name="omniwheel_x_offset" value="-0.0455" />
+    <xacro:property name="omniwheel_x_offset" value="-0.053" />
     <xacro:property name="omniwheel_vertical_offset" value="-0.01" />
     <!-- lidar Mounting Positions -->
-    <xacro:property name="lidar_x_offset" value="0.0705" />
-    <xacro:property name="lidar_vertical_offset" value="0.0807" />
+    <xacro:property name="lidar_x_offset" value="0.06155" />
+     <xacro:property name="lidar_vertical_offset" value="0.081" />
     <link name="base_link">
         <visual>
             <origin xyz="0 0 0" rpy="0 0 0" />
             <geometry>
-                <mesh filename="package://raspbot_description/meshes/base.dae" />
+                <mesh filename="package://raspbot_description/meshes/base1.dae" />
             </geometry>
         </visual>
         <collision>
-            <origin xyz="${( husky_front_bumper_extend - husky_rear_bumper_extend ) / 2.0} 0 ${base_z_size/4}" rpy="0 0 0" />
+            <origin xyz="0 0 0" rpy="0 0 0" />
             <geometry>
-                <box size="${ base_x_size + husky_front_bumper_extend + husky_rear_bumper_extend } ${base_y_size} ${base_z_size/2}"/>
+                <box size="0.01 0.01 0.01"/>
             </geometry>
         </collision>
-        <collision>
-            <origin xyz="0 0 ${base_z_size*3/4-0.01}" rpy="0 0 0" />
+        <!-- <collision>
+            <origin xyz="${base_x_size/2+0.00707} 0 0" rpy="0 0 0" />
             <geometry>
-                <box size="${base_x_size*4/5} ${base_y_size} ${base_z_size/2-0.02}"/>
+                <box size="0.0141 ${base_y_size} ${base_z_size}"/>
             </geometry>
-        </collision>
+        </collision> -->
     </link>
+    <link name="inertial_link">
+        <inertial>
+            <mass value="1.5" />
+            <origin xyz="0 0 0" />
+            <inertia ixx="0.06022" ixy="-0.002364" ixz="-0.01197" iyy="0.017386" iyz="-0.001544" izz="0.00296" />
+        </inertial>
+    </link>
+    <joint name="inertial_joint" type="fixed">
+        <origin xyz="0 0 0" rpy="0 0 0" />
+        <parent link="base_link" />
+        <child link="inertial_link" />
+    </joint>
     <link name="base_footprint"/>
     <joint name="base_footprint_joint" type="fixed">
@@ -46,26 +63,98 @@
     </joint>
     <!--  wheel  -->
-    <xacro:raspbot_wheel wheel_prefix="left">
+    <!-- <xacro:raspbot_wheel wheel_prefix="left">
         <origin xyz="${wheel_horizontal_offset} ${wheeltrack/2} ${wheel_vertical_offset}" rpy="0 0 0" />
     </xacro:raspbot_wheel>
     <xacro:raspbot_wheel wheel_prefix="right">
         <origin xyz="${wheel_horizontal_offset} ${-wheeltrack/2} ${wheel_vertical_offset}" rpy="${M_PI} 0 0" />
-    </xacro:raspbot_wheel>
+    </xacro:raspbot_wheel> -->
+    <!-- omniwheel part-->
+    <!-- <link name="omniwheel_part1_link">
+        <visual>
+            <origin xyz="0 0 0" rpy="0 0 0" />
+            <geometry>
+                <mesh filename="package://raspbot_description/meshes/omniwheel_part1.dae" />
+            </geometry>
+        </visual>
+    </link>
+    <joint name="base_omniwheel_part1_joint" type="fixed">
+        <origin xyz="${omniwheel_x_offset} 0 ${omniwheel_vertical_offset}" rpy="0 0 0" />
+        <parent link="base_link" />
+        <child link="omniwheel_part1_link" />
+    </joint> -->
+    <!-- <link name="omniwheel_part2_link">
+        <inertial>
+            <mass value="0.02" />
+            <origin xyz="0 0 0" />
+            <inertia ixx="0.001" ixy="0.001" ixz="0.001" iyy="0.001" iyz="0.001" izz="0.001" />
+        </inertial>
+        <visual>
+            <origin xyz="0 0 0" rpy="0 0 0" />
+            <geometry>
+                <mesh filename="package://raspbot_description/meshes/omniwheel_part2.dae" />
+            </geometry>
+        </visual>
+        <collision>
+            <origin xyz="0 0 0" rpy="0 0 0" />
+            <geometry>
+                <cylinder length="0.032" radius="0.028" />
+            </geometry>
+        </collision>
+    </link>
+    <joint name="omniwheel_part1_2_joint" type="continuous">
+        <origin xyz="0 0 -0.01638" rpy="0 0 0" />
+        <parent link="omniwheel_part1_link" />
+        <child link="omniwheel_part2_link" />
+        <axis xyz="0 0 1" rpy="0 0 0" />
+    </joint>
+    <link name="omniwheel_part3_link">
+        <visual>
+            <origin xyz="0 0 0" rpy="0 0 0" />
+            <geometry>
+                <mesh filename="package://raspbot_description/meshes/omniwheel_part3.dae" />
+            </geometry>
+        </visual>
+    </link>
+    <joint name="omniwheel_part2_3_joint" type="continuous">
+        <origin xyz="-0.015 0 -0.00718" rpy="0 0 0" />
+        <parent link="omniwheel_part2_link" />
+        <child link="omniwheel_part3_link" />
+        <axis xyz="0 1 0" rpy="0 0 0" />
+    </joint> -->
     <!-- omniwheel -->
-    <xacro:raspbot_omniwheel wheel_prefix="rear">
+    <!-- <xacro:raspbot_omniwheel wheel_prefix="rear">
         <origin xyz="${omniwheel_x_offset} 0 ${omniwheel_vertical_offset}" rpy="0 0 ${M_PI}" />
-    </xacro:raspbot_omniwheel>
-    <xacro:rplidar frame="lidar_link" topic="scan" robot_namespace="$(arg robot_namespace)"/>
+    </xacro:raspbot_omniwheel> -->
+    <!-- <xacro:rplidar frame="lidar_link" topic="scan" robot_namespace="$(arg robot_namespace)"/>
     <joint name="base_lidar_joint" type="fixed">
         <origin xyz="${lidar_x_offset} 0 ${lidar_vertical_offset}" rpy="0 0 0" />
         <parent link="base_link" />
         <child link="lidar_link" />
-    </joint>
+    </joint>  -->
     <!-- <link name="imu_link"/>
-    <joint name="base_footprint_joint" type="fixed">
+    <joint name="base_imu_joint" type="fixed">
         <origin xyz="0 0 0" rpy="0 0 0" />
         <parent link="base_link" />
         <child link="imu_link" />
     </joint> -->
+    <link name="test_link">
+        <visual>
+            <origin xyz="0 0 0.08" rpy="${M_PI/2} 0 0" />
+            <geometry>
+                <cylinder length="${wheel_length}" radius="${wheel_radius}" />
+            </geometry>
+        </visual>
+        <collision>
+            <origin xyz="0 0 0" rpy="0 0 0" />
+            <geometry>
+                <cylinder length="${wheel_length}" radius="${wheel_radius}" />
+            </geometry>
+        </collision>
+    </link>
+    <joint name="base_test_joint" type="fixed">
+        <origin xyz="0 0 0.08" rpy="0 0 0" />
+        <parent link="base_link" />
+        <child link="test_link" />
+    </joint>
     <!--  gazebo  -->
     <gazebo>

File: src/raspbot_description/urdf/wheel.urdf.xacro (robot description, xacro)
@@ -6,5 +6,5 @@
 				<mass value="0.167" />
 				<origin xyz="0 0 0" />
-				<inertia  ixx="0.02467" ixy="0" ixz="0" iyy="0.04411" iyz="0" izz="0.02467" />
+				<inertia  ixx="0.001" ixy="0" ixz="0" iyy="0.001" iyz="0" izz="0.001" />
 			</inertial>
             <visual>
@@ -14,4 +14,10 @@
                 </geometry>
             </visual>
+			<collision>
+				<origin xyz="0 0 0" rpy="${M_PI/2} 0 0" />
+				<geometry>
+					<cylinder length="${wheel_length}" radius="${wheel_radius}" />
+				</geometry>
+			</collision>
         </link>
         <joint name="${wheel_prefix}_wheel" type="continuous">

Commit message: change gazebo params

File: src/raspbot_description/urdf/raspbot.urdf.xacro (robot description, xacro)
@@ -27,9 +27,9 @@
     <link name="base_link">
         <inertial>
-            <mass value="2" />
-            <origin xyz="0 0 0" />
-            <inertia ixx="0.2" ixy="0" ixz="0"
-                iyy="0.2" iyz="0"
-                izz="0.2" />
+            <mass value="1.5" />
+            <origin xyz="0.0405 0 -0.0227" />
+            <inertia ixx="6.732188E-03" ixy="-5.9717E-05" ixz="-1.68616E-04"
+                iyy="1.002365E-02" iyz="1.51049E-04"
+                izz="4.991390E-03" />
         </inertial>
         <visual>
@@ -42,14 +42,11 @@
             <origin xyz="0 0 0" rpy="0 0 0" />
             <geometry>
-                <box size="0.2 0.16 0.007"/>
-                <!-- <box size="${base_x_size} ${base_y_size} ${base_z_size}"/> -->
+                <box size="${base_x_size} ${base_y_size} ${base_z_size}"/>
             </geometry>
         </collision>
         <collision>
-            <origin xyz="0.10857 0 0" rpy="0 0 0" />
-            <!-- <origin xyz="${base_x_size/2+0.00707} 0 0" rpy="0 0 0" /> -->
+            <origin xyz="${base_x_size/2+0.00707} 0 0" rpy="0 0 0" />
             <geometry>
-                <!-- <box size="0.0141 ${base_y_size} ${base_z_size}"/> -->
-                <box size="0.0141 0.16 0.007"/>
+                <box size="0.0141 ${base_y_size} ${base_z_size}"/>
             </geometry>
         </collision>
@@ -84,6 +81,5 @@
     </xacro:rplidar> -->
     <joint name="base_lidar_joint" type="fixed">
-        <!-- <origin xyz="${lidar_x_offset} 0 ${lidar_vertical_offset}" rpy="0 0 0" /> -->
-        <origin xyz="0.06155 0.0 0.081" rpy="0 0 0" />
+        <origin xyz="${lidar_x_offset} 0 ${lidar_vertical_offset}" rpy="0 0 0" />
         <parent link="base_link" />
         <child link="lidar_link" />

Commit message: alter pid params

File: src/raspbot_description/urdf/raspbot.urdf.xacro (robot description, xacro)
@@ -24,24 +24,5 @@
     <xacro:include filename="$(find raspbot_description)/urdf/rplidar.urdf.xacro" />
     <xacro:include filename="$(find raspbot_description)/urdf/omniwheel.urdf.xacro" />
-    <link name="base_footprint"/>
     <link name="base_link">
-        <inertial>
-            <!-- <mass value="2.8" /> -->
-            <!-- <mass value="1.5" /> -->
-            <mass value="1.5" />
-            <origin xyz="0.04 0.000 -0.00225" />
-            <!-- <inertia ixx="6.732188E-03" ixy="-5.9717E-05" ixz="-1.68616E-04"
-                iyy="1.002365E-02" iyz="1.51049E-04"
-                izz="4.991390E-03" /> -->
-            <!-- <inertia ixx="1.2650E-02" ixy="-1.1198E-04" ixz="-2.94157E-04"
-                iyy="1.8646767E-02" iyz="2.31768E-04"
-                izz="9.173871E-03" />     -->
-            <!-- <inertia ixx="2.2592E-02" ixy="-1.9999E-04" ixz="-5.25345E-04"
-                iyy="3.3301E-02" iyz="4.13922E-04"
-                izz="1.6383935E-02" />   -->
-            <inertia ixx="1.5" ixy="0" ixz="0"
-                iyy="1.5" iyz="0"
-                izz="1.5" />
-        </inertial>
         <visual>
             <origin xyz="0 0 0" rpy="0 0 0" />
@@ -63,8 +44,34 @@
         </collision>
     </link>
+    <link name="inertial_link">
+        <inertial>
+            <!-- <mass value="2.8" /> -->
+            <!-- <mass value="1.5" /> -->
+            <mass value="1.5" />
+            <origin xyz="0.04 0.000 -0.00225" />
+            <!-- <inertia ixx="6.732188E-03" ixy="-5.9717E-05" ixz="-1.68616E-04"
+                iyy="1.002365E-02" iyz="1.51049E-04"
+                izz="4.991390E-03" /> -->
+            <!-- <inertia ixx="1.2650E-02" ixy="-1.1198E-04" ixz="-2.94157E-04"
+                iyy="1.8646767E-02" iyz="2.31768E-04"
+                izz="9.173871E-03" />     -->
+            <!-- <inertia ixx="2.2592E-02" ixy="-1.9999E-04" ixz="-5.25345E-04"
+                iyy="3.3301E-02" iyz="4.13922E-04"
+                izz="1.6383935E-02" />   -->
+            <inertia ixx="1.5" ixy="0" ixz="0"
+                iyy="1.5" iyz="0"
+                izz="1.5" />
+        </inertial>
+    </link>
+    <joint name="base_inertial_joint" type="fixed">
+        <origin xyz="0 0 0" rpy="0 0 0" />
+        <parent link="base_link" />
+        <child link="inertial_link" />
+    </joint>
+    <link name="base_footprint"/>
     <joint name="base_footprint_joint" type="fixed">
-        <origin xyz="0 0 ${base_footprint_offset}" rpy="0 0 0" />
-        <parent link="base_footprint" />
-        <child link="base_link" />
+        <origin xyz="0 0 ${-base_footprint_offset}" rpy="0 0 0" />
+        <parent link="base_link" />
+        <child link="base_footprint" />
     </joint>
     <!--  wheel  -->
@@ -80,5 +87,5 @@
     <xacro:raspbot_omniwheel />
     <!-- <xacro:rplidar frame="lidar_link" topic="scan" robot_namespace="$(arg robot_namespace)"/> -->
-    <!-- <xacro:rplidar
+    <xacro:rplidar
         frame="lidar_link"
         topic="scan"
@@ -89,10 +96,10 @@
         sample_size="360"
         update_rate="5.5"
-        robot_namespace="$(arg robot_namespace)" /> -->
-    <!-- <joint name="base_lidar_joint" type="fixed">
+        robot_namespace="$(arg robot_namespace)" />
+    <joint name="base_lidar_joint" type="fixed">
         <origin xyz="${lidar_x_offset} 0 ${lidar_vertical_offset}" rpy="0 0 0" />
         <parent link="base_link" />
         <child link="lidar_link" />
-    </joint>  -->
+    </joint>
     <link name="imu_link"/>
     <joint name="base_imu_joint" type="fixed">

Commit message: change lidar tf

File: src/raspbot_description/urdf/raspbot.urdf.xacro (robot description, xacro)
@@ -98,5 +98,5 @@
         robot_namespace="$(arg robot_namespace)" />
     <joint name="base_lidar_joint" type="fixed">
-        <origin xyz="${lidar_x_offset} 0 ${lidar_vertical_offset}" rpy="0 0 0" />
+        <origin xyz="${lidar_x_offset} 0 ${lidar_vertical_offset}" rpy="0 0 ${M_PI}" />
         <parent link="base_link" />
         <child link="lidar_link" />
