Commit message: add depth camera D455

File: src/raspbot_description/urdf/casterwheel.urdf.xacro (robot description, xacro)
@@ -1,6 +1,6 @@
-<robot name="raspbot_omniwheel" xmlns:xacro="http://ros.org/wiki/xacro"  >
-    <xacro:macro name="raspbot_omniwheel">
-        <!-- omniwheel part-->
-        <link name="omniwheel_part1_link">
+<robot name="raspbot_casterwheel" xmlns:xacro="http://ros.org/wiki/xacro"  >
+    <xacro:macro name="raspbot_casterwheel">
+        <!-- casterwheel part-->
+        <link name="casterwheel_part1_link">
             <inertial>
                 <mass value="0.016" />
@@ -13,5 +13,5 @@
                 <origin xyz="0 0 0" rpy="0 0 0" />
                 <geometry>
-                    <mesh filename="package://raspbot_description/meshes/omniwheel_part1.dae" />
+                    <mesh filename="package://raspbot_description/meshes/casterwheel_part1.dae" />
                 </geometry>
             </visual>
@@ -23,10 +23,10 @@
             </collision>
         </link>
-        <joint name="base_omniwheel_part1_joint" type="fixed">
-            <origin xyz="${omniwheel_x_offset} 0 ${omniwheel_vertical_offset}" rpy="0 0 0" />
+        <joint name="base_casterwheel_part1_joint" type="fixed">
+            <origin xyz="${casterwheel_x_offset} 0 ${casterwheel_vertical_offset}" rpy="0 0 0" />
             <parent link="base_link" />
-            <child link="omniwheel_part1_link" />
+            <child link="casterwheel_part1_link" />
         </joint>
-        <link name="omniwheel_part2_link">
+        <link name="casterwheel_part2_link">
             <inertial>
                 <mass value="0.031" />
@@ -42,5 +42,5 @@
                 <origin xyz="0 0 0" rpy="0 0 0" />
                 <geometry>
-                    <mesh filename="package://raspbot_description/meshes/omniwheel_part2.dae" />
+                    <mesh filename="package://raspbot_description/meshes/casterwheel_part2.dae" />
                 </geometry>
             </visual>
@@ -52,11 +52,11 @@
             </collision>
         </link>
-        <joint name="omniwheel_part1_2_joint" type="continuous">
+        <joint name="casterwheel_part1_2_joint" type="continuous">
             <origin xyz="0 0 -0.01638" rpy="0 0 0" />
-            <parent link="omniwheel_part1_link" />
-            <child link="omniwheel_part2_link" />
+            <parent link="casterwheel_part1_link" />
+            <child link="casterwheel_part2_link" />
             <axis xyz="0 0 1" rpy="0 0 0" />
         </joint>
-        <link name="omniwheel_part3_link">
+        <link name="casterwheel_part3_link">
             <inertial>
                 <mass value="0.02" />
@@ -69,5 +69,5 @@
                 <origin xyz="0 0 0" rpy="0 0 0" />
                 <geometry>
-                    <mesh filename="package://raspbot_description/meshes/omniwheel_part3.dae" />
+                    <mesh filename="package://raspbot_description/meshes/casterwheel_part3.dae" />
                 </geometry>
             </visual>
@@ -79,11 +79,11 @@
             </collision>
         </link>
-        <joint name="omniwheel_part2_3_joint" type="continuous">
+        <joint name="casterwheel_part2_3_joint" type="continuous">
             <origin xyz="-0.015 0 -0.00718" rpy="0 0 0" />
-            <parent link="omniwheel_part2_link" />
-            <child link="omniwheel_part3_link" />
+            <parent link="casterwheel_part2_link" />
+            <child link="casterwheel_part3_link" />
             <axis xyz="0 1 0" rpy="0 0 0" />
         </joint>
-        <gazebo reference="omniwheel_part2_link">
+        <gazebo reference="casterwheel_part2_link">
 			<mu1 value="0.5"/>
 			<mu2 value="0.5"/>
@@ -92,5 +92,5 @@
 			<fdir1 value="1 0 0"/>
 		</gazebo>
-        <gazebo reference="omniwheel_part3_link">
+        <gazebo reference="casterwheel_part3_link">
 			<mu1 value="1"/>
 			<mu2 value="1"/>

File: src/raspbot_description/urdf/raspbot.urdf.xacro (robot description, xacro)
@@ -2,5 +2,5 @@
 <robot name="raspbot" xmlns:xacro="http://ros.org/wiki/xacro">
     <xacro:arg name="use_part_omni_model" default="true" />
-    <xacro:property name="M_PI" value="3.1415916"/>
+    <xacro:property name="M_PI" value="3.1415926535897931" />
     <!-- Base Size -->
     <xacro:property name="base_x_size" value="0.2" />
@@ -15,13 +15,17 @@
     <xacro:property name="wheel_vertical_offset" value="-0.0145" />
     <xacro:property name="wheel_horizontal_offset" value="0.068" />
-    <!-- omniWheel Mounting Positions -->
-    <xacro:property name="omniwheel_x_offset" value="-0.053" />
-    <xacro:property name="omniwheel_vertical_offset" value="-0.011" />
+    <!-- casterwheel Mounting Positions -->
+    <xacro:property name="casterwheel_x_offset" value="-0.053" />
+    <xacro:property name="casterwheel_vertical_offset" value="-0.011" />
     <!-- lidar Mounting Positions -->
     <xacro:property name="lidar_x_offset" value="0.06155" />
     <xacro:property name="lidar_vertical_offset" value="0.081" />
+    <!-- realsense D455  -->
+    <!-- Use the nominal extrinsics between camera frames if the calibrated extrinsics aren't being published. e.g. running the device in simulation  -->
+    <xacro:arg name="use_nominal_extrinsics" default="false"/>
     <xacro:include filename="$(find raspbot_description)/urdf/wheel.urdf.xacro" />
     <xacro:include filename="$(find raspbot_description)/urdf/rplidar.urdf.xacro" />
-    <xacro:include filename="$(find raspbot_description)/urdf/omniwheel.urdf.xacro" />
+    <xacro:include filename="$(find raspbot_description)/urdf/casterwheel.urdf.xacro" />
+    <xacro:include filename="$(find raspbot_description)/urdf/realsenseD455.urdf.xacro" />
     <link name="base_link">
         <visual>
@@ -84,12 +88,12 @@
         <axis xyz="0 -1 0" rpy="0 0 0" />
     </xacro:raspbot_wheel>
-    <!-- omniwheel -->
-    <xacro:raspbot_omniwheel />
+    <!-- casterwheel -->
+    <xacro:raspbot_casterwheel />
     <!-- <xacro:rplidar frame="lidar_link" topic="scan" robot_namespace="$(arg robot_namespace)"/> -->
     <xacro:rplidar
         frame="lidar_link"
         topic="scan"
-        min_angle="${-M_PI}"
-        max_angle="${M_PI}"
+        min_angle="${-M_PI/2}"
+        max_angle="${M_PI/2}"
         min_range="0.15"
         max_range="12"
@@ -108,4 +112,7 @@
         <child link="imu_link" />
     </joint>
+    <xacro:sensor_d455 parent="base_link" name="camera" use_nominal_extrinsics="$(arg use_nominal_extrinsics)">
+        <origin xyz="0.05 0 0.11" rpy="0 0 0"/>
+    </xacro:sensor_d455>
     <!--  gazebo  -->
     <gazebo>
